File: cs240lx-lab6/cs240lx-lab6.kicad_pcb (KiCad board)
At the start: 2 copper layers, 205.1 x 205.1 mm, 103 parts, among them J1 pi_zero_w, J2 oled, J3 rgb, J4 resistive_touch

Commit message: kicad files
Parts:
- removed C10, C11, C12, C13, C14, C15, C16, C17, C18, C19, C2, C20, C21, C22, C23, C24, C25, C26, C27, C28, C29, C3, C30, C31, C32, C33, C34, C35, C36, C37, C38, C39, C4, C40, C41, C42, C43, C44, C45, C46, C47, C48, C5, C6, C7, C8, C9: 100nF, Capacitor_SMD:C_0402_1005Metric_Pad0.74x0.62mm_HandSolder
- removed C49: C, Capacitor_SMD:C_0402_1005Metric_Pad0.74x0.62mm_HandSolder
- removed D1, D10, D11, D12, D13, D14, D15, D16, D17, D18, D19, D2, D20, D21, D22, D23, D24, D25, D26, D27, D28, D29, D3, D30, D31, D32, D33, D34, D35, D36, D37, D38, D39, D4, D40, D41, D42, D43, D44, D45, D46, D47, D48, D49, D5, D6, D7, D8, D9: WS2812B-2020, LED_SMD:LED_WS2812B-2020_PLCC4_2.0x2.0mm
- removed the G*** at (94.0, 118.1)
- added C51: 0.1uF, Capacitor_SMD:C_0805_2012Metric_Pad1.18x1.45mm_HandSolder, F.Cu at (258.6, 108.7)
- added COLOR: Potentiometer, Potentiometer_THT:Potentiometer_TT_P0915N, F.Cu at (193.8, 172.9)
- added DONE: SW_Push, Button_Switch_THT:SW_PUSH_6mm, F.Cu at (192.8, 133.6)
- added G***: LOGO, LOGO, F.Cu at (73.7, 123.4)
- added J5: USB_C_Receptacle_PowerOnly_6P, Connector_USB:USB_C_Receptacle_GCT_USB4125-xx-x_6P_TopMnt_Horizontal, F.Cu at (269.7, 107.7)
- added LED MODE: SW_Push, Button_Switch_THT:SW_PUSH_6mm, F.Cu at (192.8, 147.9)
- added R1: 5.1k, Resistor_SMD:R_0805_2012Metric_Pad1.20x1.40mm_HandSolder, F.Cu at (252.2, 103.1)
- added R2: 5.1k, Resistor_SMD:R_0805_2012Metric_Pad1.20x1.40mm_HandSolder, F.Cu at (249.1, 100.0)
- added R3: 1M, Resistor_SMD:R_0805_2012Metric_Pad1.20x1.40mm_HandSolder, F.Cu at (256.3, 116.3)
- added REF**: resistive_touch_correct, proj_footprints:resistive_touch_correct, F.Cu at (122.6, 127.8)
- added TP1: +3.3V, TestPoint:TestPoint_Pad_2.0x2.0mm, F.Cu at (195.6, 75.4)
- added TP2: +5V, TestPoint:TestPoint_Pad_2.0x2.0mm, F.Cu at (200.2, 75.4)
- added TP3: GND, TestPoint:TestPoint_Pad_2.0x2.0mm, F.Cu at (191.0, 75.4)
- added U1: MCP3008, proj_footprints:adc, F.Cu at (216.9, 147.5)
- C1: value 100nF -> 4.7nF; footprint Capacitor_SMD:C_0402_1005Metric_Pad0.74x0.62mm_HandSolder -> Capacitor_SMD:C_0805_2012Metric_Pad1.18x1.45mm_HandSolder
- J1: value pi_zero_w -> Raspberry_Pi_2_3; footprint Connector_PinSocket_2.54mm:PinSocket_2x20_P2.54mm_Vertical -> proj_footprints:PinSocket_2x20_P2.54mm_Vertical_rpi
- J2: value oled -> Conn_01x04_Socket; footprint Connector_PinSocket_2.54mm:PinSocket_1x04_P2.54mm_Vertical -> proj_footprints:Adafruit_SSD1306_No_Mounting_Holes_oled
- J3: value rgb -> Conn_01x03_Socket; footprint Connector_PinHeader_2.54mm:PinHeader_1x03_P2.54mm_Vertical -> proj_footprints:JST_XH_S3B-XH-A_1x03_P2.50mm_Horizontal_led
- J4: value resistive_touch -> Conn_01x06_Socket; footprint Connector_PinSocket_2.54mm:PinSocket_1x06_P2.54mm_Vertical -> proj_footprints:PinSocket_1x06_P2.54mm_Vertical_resistive_touch
- moved C1 154.2 mm to (259.6, 119.6), turned to -135 degrees
- moved J3 82.5 mm to (201.6, 58.3)
- moved J2 41.8 mm to (182.6, 98.3), turned to 0 degrees
- moved J1 34.4 mm to (240.0, 82.3)
- moved J4 25.5 mm to (85.9, 158.5), turned to 180 degrees
Connections:
- C1 pad 1: +5V -> Net-(J5-SHIELD)
- J1 pad 11: unconnected-(J1-GPIO17-Pad11) -> /gpio_17
- J1 pad 13: unconnected-(J1-GPIO27-Pad13) -> /gpio_27
- J1 pad 19: unconnected-(J1-MOSI0/GPIO10-Pad19) -> /MOSI
- J1 pad 21: unconnected-(J1-MISO0/GPIO9-Pad21) -> /MISO
- J1 pad 23: unconnected-(J1-SCLK0/GPIO11-Pad23) -> /SCLK
- J1 pad 24: unconnected-(J1-~{CE0}/GPIO8-Pad24) -> /CS
- J1 pad 32: /GPIO12 -> unconnected-(J1-PWM0/GPIO12-Pad32)
- J1 pad 40: /rgb/rgb_input -> /gpio_input
- J3 pad 1: +5V -> /gpio_input
- J3 pad 2: /rgb/rgb_input -> GND
- J3 pad 3: GND -> +5V
- J4 pad 1: /SDA -> unconnected-(J4-Pin_1-Pad1)
- J4 pad 2: /SCL -> /SDA
- J4 pad 3: GND -> /SCL
- J4 pad 4: +3.3V -> GND
- J4 pad 5: (no net) -> +3.3V
- J4 pad 6: (no net) -> unconnected-(J4-Pin_6-Pad6)
Routing:
- net +5V: track 919.2 -> 0.00 mm
- net +3.3V: track 132.4 -> 285.9 mm, vias 0 -> 1
- net /gpio_input: track 0.00 -> 97.3 mm, vias 0 -> 1
- net /gpio_27: track 0.00 -> 67.6 mm
- net /gpio_17: track 0.00 -> 55.2 mm
- net /rgb/rgb_input: track 50.3 -> 0.00 mm, vias 2 -> 0
- net /CS: track 0.00 -> 49.3 mm
- net /MOSI: track 0.00 -> 42.4 mm
- net /MISO: track 0.00 -> 40.1 mm
- net Net-(J5-SHIELD): track 0.00 -> 38.3 mm
- net /SCLK: track 0.00 -> 38.3 mm
- net /SDA: track 139.5 -> 166.8 mm
- net Net-(U1-CH0): track 0.00 -> 26.5 mm
- net Net-(J5-CC2): track 0.00 -> 21.9 mm
- net /SCL: track 140.7 -> 161.1 mm
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- added copper zone on F.Cu, net +5V
Other:
- board size 205.1 x 205.1 mm -> 254.6 x 254.6 mm
- board text added: "Aditri Patil"
- board text added: "Ashley Yumiko Raigosa"
- board text added: "B.S. Computer Science"
- board text added: "B.S. Electrical Engineering"
- board text added: "LED matrix"
- board text added: "Sally Sunmin Lee"
- board text removed: "Ashley Raigosa"
- board text removed: "Bachelor of Science Computer Science, Systems"
- board text removed: "J1"
- board text removed: "J2"
- board text removed: "J3"
- board text removed: "J4"
- board text removed: "oled"
- board text removed: "resistive_touch"
- board text removed: "rgb"
- board text removed: "rpi"
