File: cs240lx-lab6/cs240lx-lab6.kicad_sch (KiCad schematic)
At the start: 3 parts, among them J1 pi_zero_w, J2 oled, J4 resistive_touch

Commit message: kicad files
Parts:
- removed J4: resistive_touch, Connector_PinSocket_2.54mm:PinSocket_1x06_P2.54mm_Vertical, symbol Connector:Conn_01x04_Socket
- added C1: 4.7nF, Capacitor_SMD:C_0805_2012Metric_Pad1.18x1.45mm_HandSolder, symbol Device:C
- added C51: 0.1uF, Capacitor_SMD:C_0805_2012Metric_Pad1.18x1.45mm_HandSolder, symbol Device:C
- added J3: Conn_01x03_Socket, proj_footprints:JST_XH_S3B-XH-A_1x03_P2.50mm_Horizontal_led, symbol Connector:Conn_01x03_Socket
- added J4: Conn_01x06_Socket, proj_footprints:PinSocket_1x06_P2.54mm_Vertical_resistive_touch, symbol Connector:Conn_01x06_Socket
- added J5: USB_C_Receptacle_PowerOnly_6P, Connector_USB:USB_C_Receptacle_GCT_USB4125-xx-x_6P_TopMnt_Horizontal, symbol Connector:USB_C_Receptacle_PowerOnly_6P
- added R1, R2: 5.1k, Resistor_SMD:R_0805_2012Metric_Pad1.20x1.40mm_HandSolder, symbol Device:R
- added R3: 1M, Resistor_SMD:R_0805_2012Metric_Pad1.20x1.40mm_HandSolder, symbol Device:R
- added R4: Potentiometer, Potentiometer_THT:Potentiometer_TT_P0915N, symbol Simulation_SPICE:Potentiometer
- added SW1, SW2: SW_Push, Button_Switch_THT:SW_PUSH_6mm, symbol Switch:SW_Push
- added TP1: +3.3V, TestPoint:TestPoint_Pad_2.0x2.0mm, symbol Connector:TestPoint
- added TP2: +5V, TestPoint:TestPoint_Pad_2.0x2.0mm, symbol Connector:TestPoint
- added TP3: GND, TestPoint:TestPoint_Pad_2.0x2.0mm, symbol Connector:TestPoint
- added U1: MCP3008, proj_footprints:adc, symbol Analog_ADC:MCP3008
- J1: value pi_zero_w -> Raspberry_Pi_2_3; footprint Connector_PinSocket_2.54mm:PinSocket_2x20_P2.54mm_Vertical -> proj_footprints:PinSocket_2x20_P2.54mm_Vertical_rpi
- J2: value oled -> Conn_01x04_Socket; footprint Connector_PinSocket_2.54mm:PinSocket_1x04_P2.54mm_Vertical -> proj_footprints:Adafruit_SSD1306_No_Mounting_Holes_oled
Connections:
- net +3.3V: now also J4.5 (Pin_5), R4.1, TP1.1, U1.15 (Vref), U1.16 (Vdd)
- net +5V: now also C51.1, J3.3 (Pin_3), J5.A9 (VBUS), J5.B9 (VBUS), TP2.1
- net GND: now also C1.2, C51.2, J3.2 (Pin_2), J4.4 (Pin_4), J5.A12 (GND), J5.B12 (GND), R1.2, R2.2, R3.2, R4.3, SW1.2, SW2.2, TP3.1, U1.14 (AGND), U1.9 (DGND)
- net SCL: now also J4.3 (Pin_3)
- net SDA: now also J4.2 (Pin_2)
- net gpio_17: now reaches J1.11 (GPIO17)
- net gpio_17: now also SW2.1
- net gpio_27: now reaches J1.13 (GPIO27)
- net gpio_27: now also SW1.1
- net MOSI: now reaches J1.19 (MOSI0/GPIO10)
- net MOSI: now also U1.11 (Din)
- net MISO: now reaches J1.21 (MISO0/GPIO9)
- net MISO: now also U1.12 (Dout)
- net SCLK: now reaches J1.23 (SCLK0/GPIO11)
- net SCLK: now also U1.13 (CLK)
- net CS: now reaches J1.24 (~{CE0}/GPIO8)
- net CS: now also U1.10 (~{CS}/SHDN)
- net GPIO12: no longer names the net of J1.32 (PWM0/GPIO12)
- net rgb/rgb_input renamed gpio_input
- net gpio_input: now also J3.1 (Pin_1)
- new net: R4.2, U1.1 (CH0)
- new net: C1.1, J5.SH (SHIELD), R3.1
- new net: J5.A5 (CC1), R1.1
- new net: J5.B5 (CC2), R2.1
- no-connect marks 24 -> 28
Other:
- removed sheet rgb
